File: lcr-meter/CM4_GPIO.kicad_sch (KiCad schematic)
At the start: 21 parts, among them J1 Conn_01x03, J2 Conn_02x07_Odd_Even, J3 Conn_01x03, J7 Micro_SD_Card_Det, J8 THD-20-R, U18 RT9742GGJ5, U5 74LVC1G07SE-7, U9 74LVC1G07SE-7

Commit message: Progress, removal of unnecessary components
Connections:
- net Reserved: no longer Module1.76 (Reserved)
- net ETH_LEDG: no longer names the net of Module1.17 (Ethernet_nLED2(3.3v))
- net ETH_LEDY: no longer names the net of Module1.15 (Ethernet_nLED3(3.3v))
- net TRD0_N: no longer names the net of Module1.10 (Ethernet_Pair0_N)
- net TRD0_P: no longer names the net of Module1.12 (Ethernet_Pair0_P)
- net TRD1_N: no longer names the net of Module1.6 (Ethernet_Pair1_N)
- net TRD1_P: no longer names the net of Module1.4 (Ethernet_Pair1_P)
- net TRD2_N: no longer names the net of Module1.9 (Ethernet_Pair2_N)
- net TRD2_P: no longer names the net of Module1.11 (Ethernet_Pair2_P)
- net TRD3_N: no longer names the net of Module1.5 (Ethernet_Pair3_N)
- net TRD3_P: no longer names the net of Module1.3 (Ethernet_Pair3_P)
- no-connect marks 7 -> 18
Other:
- moved on the sheet: C5, D1, D2, J1, J2, J3, J7, J8, Module1A, R1, R10, R17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

Commit message: Addressable LED test board
Parts:
- Module1: Field5 2off DF40C-100DS-0.4V -> 2x DF40C-100DS-0.4V
Changed lines of the file:
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@@
 			)
 		)
-		(property "Datasheet" "https://www.diodes.com/assets/Datasheets/74LVC1G07.pdf"
+		(property "Datasheet" "http://www.ti.com/lit/sg/scyt129e/scyt129e.pdf"
 			(at 183.642 146.812 0)
 			(effects
@@
 			)
 		)
-		(property "Description" ""
+		(property "Description" "Single Buffer Gate w/ Open Drain, Low-Voltage CMOS"
 			(at 183.642 146.812 0)
 			(effects
@@
 			)
 		)
-		(property "Datasheet" "https://www.diodes.com/assets/Datasheets/74LVC1G07.pdf"
+		(property "Datasheet" "http://www.ti.com/lit/sg/scyt129e/scyt129e.pdf"
 			(at 28.194 181.61 0)
 			(effects
@@
 			)
 		)
-		(property "Description" ""
+		(property "Description" "Single Buffer Gate w/ Open Drain, Low-Voltage CMOS"
 			(at 28.194 181.61 0)
 			(effects
@@
 			)
 		)
-		(property "Description" ""
+		(property "Description" "Power symbol creates a global label with name \"GND\" , ground"
 			(at 28.194 190.5 0)
 			(effects
@@
 			)
 		)
-		(property "Description" ""
+		(property "Description" "Power symbol creates a global label with name \"GND\" , ground"
 			(at 235.204 154.94 0)
 			(effects
@@
 			)
 		)
-		(property "Field5" "2off DF40C-100DS-0.4V"
+		(property "Field5" "2x DF40C-100DS-0.4V"
 			(at 72.39 76.2 0)
 			(effects
@@
 			)
 		)
-		(property "Datasheet" "https://www.toby.co.uk/uploads/publications/1673.pdf"
+		(property "Datasheet" "~"
 			(at 157.734 48.26 0)
 			(effects
@@
 			)
 		)
-		(property "Description" ""
+		(property "Description" "Generic connector, double row, 02x20, odd/even pin numbering scheme (row 1 odd numbers, row 2 even numbers), script generated (kicad-library-utils/schlib/autogen/connector/)"
 			(at 157.734 48.26 0)
 			(effects
@@
 			)
 		)
-		(property "Datasheet" "https://search.murata.co.jp/Ceramy/image/img/A01X/G101/ENG/GRM21BR71A106KA73-01.pdf"
+		(property "Datasheet" "~"
 			(at 211.074 123.19 0)
 			(effects
@@
 			)
 		)
-		(property "Description" ""
+		(property "Description" "Unpolarized capacitor"
 			(at 211.074 123.19 0)
 			(effects
@@
 			)
 		)
-		(property "Description" ""
+		(property "Description" "Power symbol creates a global label with name \"GND\" , ground"
 			(at 166.624 74.93 0)
 			(effects
@@
 			)
 		)
-		(property "Description" ""
+		(property "Description" "Power symbol creates a global label with name \"GND\" , ground"
 			(at 151.384 74.93 0)
 			(effects
@@
 			)
 		)
-		(property "Description" ""
+		(property "Description" "Power symbol creates a global label with name \"GND\" , ground"
 			(at 38.1 149.86 0)
 			(effects
@@
 			)
 		)
-		(property "Description" ""
+		(property "Description" "Power symbol creates a global label with name \"GND\" , ground"
 			(at 101.6 149.86 0)
 			(effects
@@
 			)
 		)
-		(property "Datasheet" "http://optoelectronics.liteon.com/upload/download/DS22-2000-226/LTST-S270KGKT.pdf"
+		(property "Datasheet" "~"
 			(at 117.094 26.67 0)
 			(effects
@@
 			)
 		)
-		(property "Description" ""
+		(property "Description" "Light emitting diode"
 			(at 117.094 26.67 0)
 			(effects
@@
 			)
 		)
-		(property "Datasheet" "https://fscdn.rohm.com/en/products/databook/datasheet/passive/resistor/chip_resistor/mcr-e.pdf"
+		(property "Datasheet" "~"
 			(at 117.094 39.37 0)
 			(effects
@@
 			)
 		)
-		(property "Description" ""
+		(property "Description" "Resistor"
 			(at 117.094 39.37 0)
 			(effects
@@
 			)
 		)
-		(property "Description" ""
+		(property "Description" "Power symbol creates a global label with name \"GND\" , ground"
 			(at 183.642 154.432 0)
 			(effects
@@
 			)
 		)
-		(property "Datasheet" "http://optoelectronics.liteon.com/upload/download/DS22-2000-210/LTST-S270KRKT.pdf"
+		(property "Datasheet" "~"
 			(at 191.262 127.762 0)
 			(effects
@@
 			)
 		)
-		(property "Description" ""
+		(property "Description" "Light emitting diode"
 			(at 191.262 127.762 0)
 			(effects
@@
 			)
 		)
-		(property "Datasheet" "https://fscdn.rohm.com/en/products/databook/datasheet/passive/resistor/chip_resistor/mcr-e.pdf"
+		(property "Datasheet" "~"
 			(at 191.262 136.652 0)
 			(effects
@@
 			)
 		)
-		(property "Description" ""
+		(property "Description" "Resistor"
 			(at 191.262 136.652 0)
 			(effects
@@
 			)
 		)
-		(property "Description" ""
+		(property "Description" "Generic connector, single row, 01x03, script generated (kicad-library-utils/schlib/autogen/connector/)"
 			(at 134.366 132.08 0)
 			(effects
@@
 			)
 		)
-		(property "Description" ""
+		(property "Description" "Power symbol creates a global label with name \"GND\" , ground"
 			(at 155.956 135.89 0)
 			(effects
@@
 			)
 		)
-		(property "Datasheet" ""
+		(property "Datasheet" "~"
 			(at 186.2582 126.619 0)
 			(effects
@@
 			)
 		)
-		(property "Description" ""
+		(property "Description" "test point"
 			(at 186.2582 131.699 0)
 			(effects
@@
 			)
 		)
-		(property "Datasheet" "https://fscdn.rohm.com/en/products/databook/datasheet/passive/resistor/chip_resistor/mcr-e.pdf"
+		(property "Datasheet" "~"
 			(at 156.464 92.71 0)
 			(effects
@@
 			)
 		)
-		(property "Description" ""
+		(property "Description" "Resistor"
 			(at 156.464 92.71 0)
 			(effects
@@
 			)
 		)
-		(property "Datasheet" "https://fscdn.rohm.com/en/products/databook/datasheet/passive/resistor/chip_resistor/mcr-e.pdf"
+		(property "Datasheet" "~"
 			(at 156.464 96.52 0)
 			(effects
@@
 			)
 		)
-		(property "Description" ""
+		(property "Description" "Resistor"
 			(at 156.464 96.52 0)
 			(effects
@@
 			)
 		)
-		(property "Description" ""
+		(property "Description" "Power symbol creates a global label with name \"GND\" , ground"
 			(at 211.074 130.81 0)
 			(effects
@@
 			)
 		)
-		(property "Description" ""
+		(property "Description" "Power symbol creates a global label with name \"GND\" , ground"
 			(at 278.384 144.78 0)
 			(effects
@@
 			)
 		)
-		(property "Datasheet" "https://www.toby.co.uk/uploads/publications/1673.pdf"
+		(property "Datasheet" "~"
 			(at 71.628 173.99 0)
 			(effects
@@
 			)
 		)
-		(property "Description" ""
+		(property "Description" "Generic connector, double row, 02x07, odd/even pin numbering scheme (row 1 odd numbers, row 2 even numbers), script generated (kicad-library-utils/schlib/autogen/connector/)"
 			(at 71.628 173.99 0)
 			(effects
@@
 			)
 		)
-		(property "Description" ""
+		(property "Description" "Generic connector, single row, 01x03, script generated (kicad-library-utils/schlib/autogen/connector/)"
 			(at 123.19 132.08 0)
 			(effects
@@
 			)
 		)
-		(property "Datasheet" "https://fscdn.rohm.com/en/products/databook/datasheet/passive/resistor/chip_resistor/mcr-e.pdf"
+		(property "Datasheet" "~"
 			(at 228.854 137.16 0)
 			(effects
@@
 			)
 		)
-		(property "Description" ""
+		(property "Description" "Resistor"
 			(at 228.854 137.16 0)
 			(effects
@@
 			)
 		)
-		(property "Datasheet" ""
+		(property "Datasheet" "~"
 			(at 123.444 38.1 0)
 			(effects
@@
 			)
 		)
-		(property "Description" ""
+		(property "Description" "test point"
 			(at 123.444 33.02 0)
 			(effects
@@
 			)
 		)
-		(property "Datasheet" "https://fscdn.rohm.com/en/products/databook/datasheet/passive/resistor/chip_resistor/mcr-e.pdf"
+		(property "Datasheet" "~"
 			(at 273.939 153.67 0)
 			(effects
@@
 			)
 		)
-		(property "Description" ""
+		(property "Description" "Resistor"
 			(at 273.939 153.67 0)
 			(effects
@@
 			)
 		)
-		(property "Datasheet" "https://fscdn.rohm.com/en/products/databook/datasheet/passive/resistor/chip_resistor/mcr-e.pdf"
+		(property "Datasheet" "~"
 			(at 228.854 144.78 0)
 			(effects
@@
 			)
 		)
-		(property "Description" ""
+		(property "Description" "Resistor"
 			(at 228.854 144.78 0)
 			(effects
