File: lcr-meter/lcd.kicad_sch (KiCad schematic)
At the start: 1 part, among them U4 CR2013-MI2120

Commit message: Schematic polishing
Other:
- note added: "Should not need decoupling or any external components."
Changed lines of the file:
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@@
+		)
+	)
+	(text "Should not need decoupling or any external components."
+		(exclude_from_sim no)
+		(at 158.75 113.538 0)
+		(effects
+			(font
+				(size 1.27 1.27)
+			)
 		)
 	)
