File: lcr-meter/lcr-meter.kicad_sch (KiCad schematic)
At the start: 4 parts

Commit message: PCB updates
Other:
- note added: "LAYOUT FIXES NEEDED - Change position of the Poewr switch. Unassembleable in current state."
- note added: "SCHEMATIC FIXES NEEDED X Change Sense MUX footrpints X Chnage User input button schematic X Fix LCD interface - REMOVE EXT ADC? X Add 1 nF Capacitor in parallel with sine gen buffer amp X Add 20 pF Capacitor to output of AD9833 X Swap zero Ohm resistors with jumpers"

Commit message: REV B order submitted
Connections:
- no-connect marks 0 -> 1
Other:
- removed sheet ADC
- sheet MCU ports: added none; removed MCP3202_NCS
- note added: "LAYOUT FIXES NEEDED X Change position of the Poewr switch. Unassembleable in current state."
- note added: "SCHEMATIC FIXES NEEDED X Change Sense MUX footrpints X Chnage User input button schematic X Fix LCD interface X REMOVE EXT ADC? X Add 1 nF Capacitor in parallel with sine gen buffer amp X Add 20 pF Capacitor to output of AD9833 X Swap zero Ohm resistors with jumpers"
- note removed: "LAYOUT FIXES NEEDED - Change position of the Poewr switch. Unassembleable in current state."
- note removed: "SCHEMATIC FIXES NEEDED X Change Sense MUX footrpints X Chnage User input button schematic X Fix LCD interface - REMOVE EXT ADC? X Add 1 nF Capacitor in parallel with sine gen buffer amp X Add 20 pF Capacitor to output of AD9833 X Swap zero Ohm resistors with jumpers"

Commit message: Polishing, Poster Creation
Other:
- sheet DAC renamed Sine Generator
- sheet MCU: file stm32f469vit.kicad_sch -> stm32f446re.kicad_sch
- sheet Sensing ports: added +1V8, +3V3, +5V, -5V; removed none
- sheet Sine Generator ports: added +3V3, +5V, -5V; removed none
- note added: "AD9833 + PA"
- note added: "Buck Converters + Linear Regulators"
- note added: "LCD"
- note added: "MUX + Differential Amplifiers DUT Measurement"
- note added: "STM32F446RE"
- note removed: "DONE"
- note removed: "LAYOUT FIXES NEEDED X Change position of the Poewr switch. Unassembleable in current state."
- note removed: "SCHEMATIC FIXES NEEDED X Change Sense MUX footrpints X Chnage User input button schematic X Fix LCD interface X REMOVE EXT ADC? X Add 1 nF Capacitor in parallel with sine gen buffer amp X Add 20 pF Capacitor to output of AD9833 X Swap zero Ohm resistors with jumpers"
