File: lcr-meter/dac.kicad_sch (KiCad schematic)
At the start: 9 parts, among them U1 KC2016Z20.0000C15XXK, U19 AD9833xRM, U20 LF353N/NOPB

Commit message: PCB updates
Parts:
- added C10: 20p, Capacitor_SMD:C_0402_1005Metric, symbol Device:C_Small
- added C11, C21: 100n, Capacitor_SMD:C_0402_1005Metric, symbol Device:C_Small
- added C52: 10n, Capacitor_SMD:C_0402_1005Metric, symbol Device:C_Small
Connections:
- net +5V: now also C11.1
- net -5V: now also C21.1
- net GND: now also C10.2, C11.2, C21.2
- net I_OUT: now also C52.2
- net Signal: now also C10.1
- net at R22.1, R7.1, U20.2 (IN-): now also C52.1
Other:
- note added: "Pin Compatible wiht LM833N"
- note added: "This cap was needed (Found experimentally) for some reason"
- note removed: "REPLACE WITH LM833N, ADD x2 GAIN LM833N is discontinued; I am using a LF353N instead. This new opamp has lower GBWP (lm833n = 15MHz, lf353N = 4 MHz), but higher slew rate (lm833n = 7v/us, lf353n = 13v/us). Datasheet says that minimum recommended supply is +-6V, but says it may work with a lower supply (with lowered GBWP and slew rate) Check this with the breadboard circuit first before continuing."
- moved on the sheet: C43, R22, R7, U20A, U20B
